File: TTuaefi.kicad_sch (KiCad schematic)
At the start: 72 parts, among them J1 Conn_02x02_Odd_Even, J10 5569-16A2, J11 Conn_02x02_Odd_Even, J12 Conn_02x02_Odd_Even, J13 Conn_02x02_Odd_Even, J14 Conn_02x02_Odd_Even, J15 Conn_02x02_Odd_Even, J16 Conn_02x02_Odd_Even, J17 Conn_02x02_Odd_Even, J18 Conn_02x02_Odd_Even, J19 Conn_02x02_Odd_Even, J2 5569-20A2, J20 Conn_02x02_Odd_Even, J21 Conn_02x02_Odd_Even, J22 Conn_02x02_Odd_Even, J24 Conn_02x02_Odd_Even, J3 5569-06A2, J4 5569-08A2, J5 5569-18A2, J6 Conn_01x06, J7 Conn_01x05_Male, J8 USB_B_Mini, J9 USB_C, M1 Module-power_12and5V-0.3, M2 Module-knock-0.2, M3 Module-vr-discrete-0.5, M4 Module-vr-max9924-0.1, M5 Module-wbo-0.5, M6 Module:mega-mcu100/0.3, M7 Module-can-0.1, P1 Pad, P2 Pad, P3 Pad, P4 Pad, P5 Pad, P6 Pad, P7 Pad, P8 Pad, U5 JDY-33

Commit message: Update TTuaefi.kicad_sch
Other:
- title: UAEFI -> TTuaefi
Changed lines of the file:
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@@
 	(paper "A3" portrait)
 	(title_block
-		(title "UAEFI")
+		(title "TTuaefi")
 		(date "2025-04-30")
-		(rev "E")
+		(rev "a")
 		(company "rusEFI.com")
 		(comment 1 "https://rusefi.com/s/uaefi")
